Commit message: adding robot arm

File: src/my_robot_description/urdf/arm.xacro (robot description, xacro)
@@ -97,5 +97,5 @@
         <origin xyz="0 0 0.05087" rpy="0 0 0" />
         <axis xyz="0 0 1" />
-        <limit effort="1000.0" velocity="1.0" lower="-2.356" upper="2.356" />
+        <limit effort="1000.0" velocity="1.0" lower="-1.57" upper="1.57" />
     </joint>
     <joint name="joint2" type="revolute">
@@ -118,5 +118,5 @@
         <origin xyz="0 0 0.09795" rpy="0 0 0" />
         <axis xyz="0 0 1" />
-        <limit effort="1000.0" velocity="1.0" lower="-3.14" upper="3.14" />
+        <limit effort="1000.0" velocity="1.0" lower="-1.57" upper="1.57" />
     </joint>
     <joint name="joint5" type="revolute">

File: src/my_robot_description/urdf/my_robot.urdf.xacro (robot description, xacro)
@@ -3,3 +3,9 @@
     <xacro:include filename="common_properties.xacro" />
     <xacro:include filename="arm.xacro" />
+    <xacro:include filename="gripper.xacro" />
+    <joint name="gripper_base_joint" type="fixed">
+        <parent link="tool_link" />
+        <child link="gripper_base_link" />
+        <origin xyz="0 0 0" rpy="0 0 0" />
+    </joint>
 </robot>

File: src/my_robot_moveit_config/config/my_robot.ros2_control.xacro (robot description, xacro)
@@ -7,5 +7,5 @@
                 <!-- By default, set up controllers for simulation. This won't work on real hardware -->
                 <plugin>mock_components/GenericSystem</plugin>
-\            </hardware>
+            </hardware>
             <joint name="joint1">
                 <command_interface name="position"/>
@@ -38,4 +38,10 @@
                 </state_interface>
             </joint>
+            <joint name="gripper_left_finger_joint">
+                <command_interface name="position"/>
+                <state_interface name="position">
+                  <param name="initial_value">${initial_positions['gripper_left_finger_joint']}</param>
+                </state_interface>
+            </joint>
         </ros2_control>
     </xacro:macro>

Commit message: push

File: src/my_robot_description/urdf/arm.xacro (robot description, xacro)
@@ -79,14 +79,14 @@
         <visual>
             <geometry>
-                <box size="0.02177 0.02177 0.00299" />
+                <box size="0.02177 0.02177 0.01999" />
             </geometry>
-            <origin xyz="0 0 0.001495" rpy="0 0 0" />
+            <origin xyz="0 0 0.009995" rpy="0 0 0" />
             <material name="blue" />
         </visual>
         <collision>
             <geometry>
-                <box size="0.02177 0.02177 0.00299" />
+                <box size="0.02177 0.02177 0.01099" />
             </geometry>
-            <origin xyz="0 0 0.001495" rpy="0 0 0" />
+            <origin xyz="0 0 0.009995" rpy="0 0 0" />
         </collision>
     </link>
@@ -130,5 +130,5 @@
         <parent link="wrist_link" />
         <child link="tool_link" />
-        <origin xyz="0 0 0.00299" rpy="0 0 0" />
+        <origin xyz="0 0 0.009995" rpy="0 0 0" />
     </joint>
 </robot>

File: src/my_robot_description/urdf/my_robot.urdf.xacro (robot description, xacro)
@@ -3,4 +3,5 @@
     <xacro:include filename="common_properties.xacro" />
     <xacro:include filename="arm.xacro" />
+    <xacro:include filename="my_robot.ros2_control.xacro" />
     <xacro:include filename="gripper.xacro" />
     <joint name="gripper_base_joint" type="fixed">
