Commit message: Revert "Fix integration issues between web bridge, MoveIt, and hardware."
This reverts commit d2cdc02d8e1688b0683cb72bc4b2e08b0b04b532.

File: my_robot_description/urdf/my_robot.urdf.xacro (robot description, xacro)
@@ -1,13 +1,8 @@
 <?xml version="1.0"?>
 <robot name="my_robot" xmlns:xacro="http://www.ros.org/wiki/xacro">
-    <xacro:arg name="use_mock_hardware" default="true"/>
-    <xacro:arg name="serial_port" default="/dev/ttyUSB0"/>
-    <xacro:arg name="baud_rate" default="115200"/>
-    <xacro:arg name="initial_positions_file"
-               default="$(find my_robot_description)/config/initial_positions.yaml"/>
     <xacro:include filename="common_properties.xacro" />
     <xacro:include filename="arm.xacro" />
+    <xacro:include filename="my_robot.ros2_control.xacro" />
     <xacro:include filename="gripper.xacro" />
-    <xacro:include filename="my_robot.ros2_control.xacro" />
     <joint name="gripper_base_joint" type="fixed">
         <parent link="tool_link" />
@@ -15,9 +10,3 @@
         <origin xyz="0 0 0" rpy="0 0 0" />
     </joint>
-    <xacro:my_robot_ros2_control
-        name="ArmSystem"
-        use_mock_hardware="$(arg use_mock_hardware)"
-        serial_port="$(arg serial_port)"
-        baud_rate="$(arg baud_rate)"
-        initial_positions_file="$(arg initial_positions_file)" />
 </robot>

File: my_robot_moveit_config/config/my_robot.ros2_control.xacro (robot description, xacro)
@@ -1,18 +1,15 @@
 <?xml version="1.0"?>
 <robot xmlns:xacro="http://www.ros.org/wiki/xacro">
-        <ros2_control name="Arm" type="system">
+    <xacro:macro name="my_robot_ros2_control" params="name initial_positions_file">
+        <xacro:property name="initial_positions" value="${xacro.load_yaml(initial_positions_file)['initial_positions']}"/>
+        <ros2_control name="${name}" type="system">
             <hardware>
                 <!-- By default, set up controllers for simulation. This won't work on real hardware -->
                 <plugin>mock_components/GenericSystem</plugin>
-                <!-- For real hardware, use the custom hardware interface -->
-                <!-- <plugin>arm_hardware/ArmHardware</plugin>
-                <param name="serial_device">/dev/ttyUSB0</param>
-                <param name="baud_rate">115200</param>
-                 -->
             </hardware>
             <joint name="joint1">
                 <command_interface name="position"/>
                 <state_interface name="position">
-                  <param name="initial_value">0.0</param>
+                  <param name="initial_value">${initial_positions['joint1']}</param>
                 </state_interface>
             </joint>
@@ -20,5 +17,5 @@
                 <command_interface name="position"/>
                 <state_interface name="position">
-                  <param name="initial_value">0.0</param>
+                  <param name="initial_value">${initial_positions['joint2']}</param>
                 </state_interface>
             </joint>
@@ -26,5 +23,5 @@
                 <command_interface name="position"/>
                 <state_interface name="position">
-                  <param name="initial_value">0.0</param>
+                  <param name="initial_value">${initial_positions['joint3']}</param>
                 </state_interface>
             </joint>
@@ -32,5 +29,5 @@
                 <command_interface name="position"/>
                 <state_interface name="position">
-                  <param name="initial_value">0.0</param>
+                  <param name="initial_value">${initial_positions['joint4']}</param>
                 </state_interface>
             </joint>
@@ -38,5 +35,5 @@
                 <command_interface name="position"/>
                 <state_interface name="position">
-                  <param name="initial_value">0.0</param>
+                  <param name="initial_value">${initial_positions['joint5']}</param>
                 </state_interface>
             </joint>
@@ -44,7 +41,8 @@
                 <command_interface name="position"/>
                 <state_interface name="position">
-                  <param name="initial_value">0.0</param>
+                  <param name="initial_value">${initial_positions['gripper_left_finger_joint']}</param>
                 </state_interface>
             </joint>
         </ros2_control>
+    </xacro:macro>
 </robot>

File: my_robot_moveit_config/config/my_robot.urdf.xacro (robot description, xacro)
@@ -1,9 +1,9 @@
 <?xml version="1.0"?>
 <robot xmlns:xacro="http://www.ros.org/wiki/xacro" name="my_robot">
-    <xacro:arg name="use_mock_hardware" default="true"/>
-    <xacro:arg name="serial_port" default="/dev/ttyUSB0"/>
-    <xacro:arg name="baud_rate" default="115200"/>
-    <xacro:arg name="initial_positions_file"
-               default="$(find my_robot_moveit_config)/config/initial_positions.yaml"/>
+    <xacro:arg name="initial_positions_file" default="initial_positions.yaml" />
+    <!-- Import my_robot urdf file -->
     <xacro:include filename="$(find my_robot_description)/urdf/my_robot.urdf.xacro" />
+    <!-- Import control_xacro -->
+    <xacro:include filename="my_robot.ros2_control.xacro" />
+    <xacro:my_robot_ros2_control name="FakeSystem" initial_positions_file="$(arg initial_positions_file)"/>
 </robot>
